Commit message: added diff_drive

File: urdf/combined.urdf (robot description, URDF)
Before this commit: robot hitomi, 10 links, 9 joints
Links:
- added link camera_link, mass 0.01; collision cylinder length=0.01 radius=0.01; visual cylinder length=0.01 radius=0.01
- link display_link: geometry collision box size=0.01 0.08 0.03; visual box size=0.01 0.08 0.03
Joints:
- added joint camera_joint: type fixed, parent chassis_link, child camera_link, origin xyz=0.128 0 0.08
- joint leg_fl_joint: origin xyz=0.15 -0.9 0.15 rpy=0 0 0 -> xyz=0.15 0.09 0.03 rpy=0 0 0
- joint leg_fr_joint: origin xyz=1.5 0.9 1.5 rpy=0 0 0 -> xyz=0.15 -0.09 0.03 rpy=0 0 0
- joint leg_rl_joint: origin xyz=-1.5 -0.9 1.5 rpy=0 0 0 -> xyz=-0.15 0.09 0.03 rpy=0 0 0
- joint leg_rr_joint: origin xyz=-1.5 0.9 1.5 rpy=0 0 0 -> xyz=-0.15 -0.09 0.03 rpy=0 0 0
- joint wheel_fl_joint: axis 0 0 1 -> 0 1 0 ; origin xyz=0.08 -0.02 -0.05 -> xyz=0.08 0.02 -0.05
- joint wheel_fr_joint: axis 0 0 1 -> 0 1 0 ; origin xyz=0.8 0.2 -0.5 -> xyz=0.08 -0.02 -0.05
- joint wheel_rl_joint: axis 0 0 1 -> 0 1 0 ; origin xyz=-0.8 -0.2 -0.5 -> xyz=-0.08 0.02 -0.05
- joint wheel_rr_joint: axis 0 0 1 -> 0 1 0 ; origin xyz=-0.8 0.2 -0.5 -> xyz=-0.08 -0.02 -0.05

File: urdf/gazebo_plugins.urdf.xacro (robot description, xacro)
@@ -7,3 +7,31 @@
     </plugin>
   </gazebo>
+  <gazebo>
+    <plugin filename="gz-sim-diff-drive-system" name="gz::sim::systems::DiffDrive">
+        <left_joint>wheel_fl_joint</left_joint>
+        <right_joint>wheel_fr_joint</right_joint>
+        <wheel_separation>0.220334</wheel_separation>
+        <wheel_radius>0.02</wheel_radius>
+        <max_linear_acceleration>5i</max_linear_acceleration>
+        <odom_publish_frequency>100</odom_publish_frequency>
+        <topic>cmd_vel</topic>
+        <odom_topic>odom</odom_topic>
+    </plugin>
+</gazebo>
+<gazebo reference="wheel_fl">
+  <mu1>1.0</mu1>
+  <mu2>1.0</mu2>
+</gazebo>
+<gazebo reference="wheel_fr">
+  <mu1>1.0</mu1>
+  <mu2>1.0</mu2>
+</gazebo>
+<gazebo reference="wheel_rl">
+  <mu1>0.000001</mu1>
+  <mu2>0.000001</mu2>
+</gazebo>
+<gazebo reference="wheel_rr">
+  <mu1>0.000001</mu1>
+  <mu2>0.000001</mu2>
+</gazebo>
 </robot>

File: urdf/wheels.urdf.xacro (robot description, xacro)
@@ -16,5 +16,5 @@
             </collision>
             <inertial>
-                <mass value="0.5" />
+                <mass value="0.05" />
                 <inertia ixx="0.005" ixy="0" ixz="0" iyy="0.005" iyz="0" izz="0.005" />
               </inertial>
@@ -24,5 +24,5 @@
             <child link="wheel_${suffix}"/>
             <origin xyz="${xyz}"/>
-            <axis xyz="0 0 1"/>
+            <axis xyz="0 1 0 "/>
         </joint>
     </xacro:macro>
