Commit message: updated the urdf

File: urdf/chassis.urdf.xacro (robot description, xacro)
@@ -1,7 +1,8 @@
 <?xml version="1.0"?>
-<robot name="hitomi" xmlns:xacro="https://ros.org/wiki/xacro">
+<robot  xmlns:xacro="http://ros.org/wiki/xacro">
     <xacro:macro name="chassis">
         <link name="chassis_link">
             <visual>
+                <origin xyz="0 0 0.77" rpy="0 0 0"/>
                 <geometry>
                     <mesh filename="package://hitomi/meshes/body.dae"/>
@@ -12,4 +13,5 @@
             </visual>
             <collision>
+                <origin xyz="0 0 0" rpy="0 0 0"/>
                 <geometry>
                     <mesh filename="package://hitomi/meshes/body.stl"/>
@@ -24,4 +26,19 @@
               </inertial>
         </link>
+        <link name="display_link">
+            <visual>
+                <origin xyz="0.7 0 2.5" rpy="0 0 0"/>
+                <geometry>
+                    <box size="0.1 0.8 0.3"/>
+                </geometry>
+                <material name="white">
+                    <color rgba="1 1 1 1"/>
+                </material>
+            </visual>
+        </link>
+        <joint name="display_joint" type="fixed">
+            <parent link="chassis_link"/>
+            <child link="display_link"/>
+        </joint>
     </xacro:macro>
 </robot>

File: urdf/wheels.urdf.xacro (robot description, xacro)
@@ -6,10 +6,10 @@
                 <origin xyz="0 0 0" rpy="1.570795 0 0"/>
                 <geometry>
-                    <cyinder radius="0.2" length="0.2"/>
+                    <cylinder radius="0.2" length="0.2"/>
                 </geometry>
             </visual>
             <collision>
                 <geometry>
-                    <cylinder radius="${wheel_rad}" length="${wheel_wid}"/>
+                    <cylinder radius="0.2" length="0.2"/>
                 </geometry>
             </collision>

Commit message: checking another branch

File: urdf/chassis.urdf.xacro (robot description, xacro)
@@ -2,4 +2,5 @@
 <robot  xmlns:xacro="http://ros.org/wiki/xacro">
     <xacro:macro name="chassis">
+        <link name="base_footprint"/>
         <link name="chassis_link">
             <visual>
@@ -26,4 +27,8 @@
               </inertial>
         </link>
+        <joint name="base_joint" type="fixed">
+            <parent link="base_footprint"/>
+            <child link="chassis_link"/>
+        </joint>
     </xacro:macro>
 </robot>

File: urdf/combined.urdf (robot description, URDF)
Before this commit: robot hitomi, 11 links, 10 joints
Links:
- removed link display_link
- added link lidar_link; visual cylinder length=0.02 radius=0.02
- link wheel_fl: mass 0.5 -> 0.05
- link wheel_fr: mass 0.5 -> 0.05
- link wheel_rl: mass 0.5 -> 0.05
- link wheel_rr: mass 0.5 -> 0.05
Joints:
- removed joint display_joint
- added joint lidar_joint: type fixed, parent chassis_link, child lidar_link, origin xyz=0.07 0 0.12 rpy=0 0 0

File: urdf/combined.urdf.xacro (robot description, xacro)
@@ -4,5 +4,5 @@
     <xacro:include filename="$(find hitomi)/urdf/legs.urdf.xacro"/>
     <xacro:include filename="$(find hitomi)/urdf/wheels.urdf.xacro"/>
-    <xacro:include filename="$(find hitomi)/urdf/display.urdf.xacro"/>
+    <xacro:include filename="$(find hitomi)/urdf/lidar.urdf.xacro"/>
     <xacro:include filename="$(find hitomi)/urdf/camera.urdf.xacro"/>
     <xacro:include filename="$(find hitomi)/urdf/gazebo_plugins.urdf.xacro"/>
@@ -16,5 +16,5 @@
     <xacro:wheel suffix="rl" parent="leg_rl" xyz="-0.08 0.02 -0.05" />
     <xacro:wheel suffix="rr" parent="leg_rr" xyz="-0.08 -0.02 -0.05" />
-    <xacro:display xyz="0.07 0 0.11" />
+    <xacro:lidar xyz="0.07 0 0.12" />
     <xacro:camera/>
 </robot>

File: urdf/gazebo_plugins.urdf.xacro (robot description, xacro)
@@ -13,9 +13,18 @@
         <wheel_separation>0.220334</wheel_separation>
         <wheel_radius>0.02</wheel_radius>
-        <max_linear_acceleration>5i</max_linear_acceleration>
-        <odom_publish_frequency>100</odom_publish_frequency>
-        <topic>cmd_vel</topic>
+        <max_linear_acceleration>5</max_linear_acceleration>
+        <odom_publish_frequency>30</odom_publish_frequency>
         <odom_topic>odom</odom_topic>
+        <!--odometry_source>world</odometry_source>
+        <tf_topic>tf</tf_topic>
+        <frame_id>odom</frame_id>
+        <child_frame_id>base_footprint</child_frame_id>
+        <publish_odom>true</publish_odom>
+        <publish_odom_tf>true</publish_odom_tf-->
     </plugin>
+  <!--plugin filename="gz-sim-joint-state-publisher-system"
+  name="gz::sim::systems::JointStatePublisher">
+      <topic>joint_states</topic>
+  </plugin-->
 </gazebo>
 <gazebo reference="wheel_fl">
