Commit message: added camera

File: urdf/camera.urdf.xacro (robot description, xacro)
@@ -2,4 +2,51 @@
 <robot xmlns:xacro="http://ros.org/wiki/xacro">
 <xacro:macro name="camera">
+    <link name="camera_link">
+        <visual>
+            <origin xyz="0 0 0" rpy="0 1.570795 0"/>
+            <geometry>
+                <cylinder radius="0.01" length="0.01"/>
+            </geometry>
+            <material name="black">
+                <color rgba="0 0 0 1"/>
+            </material>
+        </visual>
+        <collision>
+            <geometry>
+                <cylinder radius="0.01" length="0.01"/>
+            </geometry>
+        </collision>
+        <inertial>
+            <mass value="0.01"/>
+            <inertia ixx="0.005" ixy="0" ixz="0" iyy="0.005" iyz="0" izz="0.005" />
+            <origin xyz="0 0 0" rpy="0 0 0"/>
+        </inertial>
+    </link>
+    <joint name="camera_joint" type="fixed">
+        <parent link="chassis_link"/>
+        <child link="camera_link"/>
+        <origin xyz="0.128 0 0.08"/>
+    </joint>
+    <gazebo reference="camera_link">
+     <sensor name="camera_fr" type="camera">
+        <pose>-0.005 0 0 0 0 0</pose>
+        <always_on>true</always_on>
+        <update_rate>30</update_rate>
+        <visualize>true</visualize>
+        <topic>camera/image_raw</topic>
+        <camera>
+          <camera_info_topic>/camera_info</camera_info_topic>
+          <horizontal_fov>1.5</horizontal_fov>
+          <image>
+            <width>640</width>
+            <height>480</height>
+          </image>
+          <clip>
+            <near>0.01</near>
+            <far>300</far>
+          </clip>
+        </camera>
+      </sensor>
+    </gazebo>
 </xacro:macro>
 </robot>

File: urdf/chassis.urdf.xacro (robot description, xacro)
@@ -4,5 +4,5 @@
         <link name="chassis_link">
             <visual>
-                <origin xyz="0 0 0.77" rpy="0 0 0"/>
+                <origin xyz="0 0 0.07" rpy="0 0 0"/>
                 <geometry>
                     <mesh filename="package://hitomi/meshes/body.dae"/>
@@ -13,5 +13,5 @@
             </visual>
             <collision>
-                <origin xyz="0 0 0" rpy="0 0 0"/>
+                <origin xyz="0 0 0.07" rpy="0 0 0"/>
                 <geometry>
                     <mesh filename="package://hitomi/meshes/body.stl"/>
@@ -26,19 +26,4 @@
               </inertial>
         </link>
-        <link name="display_link">
-            <visual>
-                <origin xyz="0.7 0 2.5" rpy="0 0 0"/>
-                <geometry>
-                    <box size="0.1 0.8 0.3"/>
-                </geometry>
-                <material name="white">
-                    <color rgba="1 1 1 1"/>
-                </material>
-            </visual>
-        </link>
-        <joint name="display_joint" type="fixed">
-            <parent link="chassis_link"/>
-            <child link="display_link"/>
-        </joint>
     </xacro:macro>
 </robot>

File: urdf/combined.urdf.xacro (robot description, xacro)
@@ -4,12 +4,17 @@
     <xacro:include filename="$(find hitomi)/urdf/legs.urdf.xacro"/>
     <xacro:include filename="$(find hitomi)/urdf/wheels.urdf.xacro"/>
+    <xacro:include filename="$(find hitomi)/urdf/display.urdf.xacro"/>
+    <xacro:include filename="$(find hitomi)/urdf/camera.urdf.xacro"/>
+    <xacro:include filename="$(find hitomi)/urdf/gazebo_plugins.urdf.xacro"/>
     <xacro:chassis/>
-    <xacro:leg suffix="fl" parent="chassis_link" xyz="1.5 -0.9 1.5" rpy="0 0.523 0"/>
-    <xacro:leg suffix="fr" parent="chassis_link" xyz="1.5 0.9 1.5" rpy="0 0.523 0"/>
-    <xacro:leg suffix="rl" parent="chassis_link" xyz="-1.5 -0.9 1.5" rpy="0 -0.523 0"/>
-    <xacro:leg suffix="rr" parent="chassis_link" xyz="-1.5 0.9 1.5" rpy="0 -0.523 0"/>
-    <xacro:wheel suffix="fl" parent="leg_fl" xyz="0.8 -0.2 -0.5" />
-    <xacro:wheel suffix="fr" parent="leg_fr" xyz="0.8 0.2 -0.5" />
-    <xacro:wheel suffix="rl" parent="leg_rl" xyz="-0.8 -0.2 -0.5" />
-    <xacro:wheel suffix="rr" parent="leg_rr" xyz="-0.8 0.2 -0.5" />
+    <xacro:leg suffix="fl" parent="chassis_link" xyz="0.15 0.09 0.03" rpy="0 0.523 0"/>
+    <xacro:leg suffix="fr" parent="chassis_link" xyz="0.15 -0.09 0.03" rpy="0 0.523 0"/>
+    <xacro:leg suffix="rl" parent="chassis_link" xyz="-0.15 0.09 0.03" rpy="0 -0.523 0"/>
+    <xacro:leg suffix="rr" parent="chassis_link" xyz="-0.15 -0.09 0.03" rpy="0 -0.523 0"/>
+    <xacro:wheel suffix="fl" parent="leg_fl" xyz="0.08 0.02 -0.05"/>
+    <xacro:wheel suffix="fr" parent="leg_fr" xyz="0.08 -0.02 -0.05"/>
+    <xacro:wheel suffix="rl" parent="leg_rl" xyz="-0.08 0.02 -0.05" />
+    <xacro:wheel suffix="rr" parent="leg_rr" xyz="-0.08 -0.02 -0.05" />
+    <xacro:display xyz="0.07 0 0.11" />
+    <xacro:camera/>
 </robot>

File: urdf/legs.urdf.xacro (robot description, xacro)
@@ -13,4 +13,5 @@
             </visual>
             <collision>
+                <origin xyz="0 0 0" rpy="${rpy}"/>
                 <geometry>
                     <mesh filename="package://hitomi/meshes/leg.stl"/>

File: urdf/wheels.urdf.xacro (robot description, xacro)
@@ -6,10 +6,11 @@
                 <origin xyz="0 0 0" rpy="1.570795 0 0"/>
                 <geometry>
-                    <cylinder radius="0.2" length="0.2"/>
+                    <cylinder radius="0.02" length="0.02"/>
                 </geometry>
             </visual>
             <collision>
+                <origin xyz="0 0 0" rpy="1.570795 0 0"/>
                 <geometry>
-                    <cylinder radius="0.2" length="0.2"/>
+                    <cylinder radius="0.02" length="0.02"/>
                 </geometry>
             </collision>

Commit message: adjusted

File: urdf/camera.urdf.xacro (robot description, xacro)
@@ -26,5 +26,5 @@
         <parent link="chassis_link"/>
         <child link="camera_link"/>
-        <origin xyz="0.128 0 0.08"/>
+        <origin xyz="0.125 0 0.08"/>
     </joint>
     <gazebo reference="camera_link">

File: urdf/chassis.urdf.xacro (robot description, xacro)
@@ -7,5 +7,5 @@
                 <origin xyz="0 0 0.07" rpy="0 0 0"/>
                 <geometry>
-                    <mesh filename="package://hitomi/meshes/body.dae"/>
+                    <mesh filename="package://hitomi_display/meshes/body.dae"/>
                 </geometry>
                 <material name="true_turquoise">
@@ -16,5 +16,5 @@
                 <origin xyz="0 0 0.07" rpy="0 0 0"/>
                 <geometry>
-                    <mesh filename="package://hitomi/meshes/body.stl"/>
+                    <mesh filename="package://hitomi_display/meshes/body.stl"/>
                 </geometry>
             </collision>

File: urdf/combined.urdf.xacro (robot description, xacro)
@@ -1,9 +1,9 @@
 <?xml version="1.0"?>
-<robot name="hitomi" xmlns:xacro="https://ros.org/wiki/xacro">
-    <xacro:include filename="$(find hitomi)/urdf/chassis.urdf.xacro"/>
-    <xacro:include filename="$(find hitomi)/urdf/legs.urdf.xacro"/>
-    <xacro:include filename="$(find hitomi)/urdf/wheels.urdf.xacro"/>
-    <xacro:include filename="$(find hitomi)/urdf/lidar.urdf.xacro"/>
-    <xacro:include filename="$(find hitomi)/urdf/camera.urdf.xacro"/>
+<robot name="hitomi_display" xmlns:xacro="https://ros.org/wiki/xacro">
+    <xacro:include filename="$(find hitomi_display)/urdf/chassis.urdf.xacro"/>
+    <xacro:include filename="$(find hitomi_display)/urdf/legs.urdf.xacro"/>
+    <xacro:include filename="$(find hitomi_display)/urdf/wheels.urdf.xacro"/>
+    <xacro:include filename="$(find hitomi_display)/urdf/display.urdf.xacro"/>
+    <xacro:include filename="$(find hitomi_display)/urdf/camera.urdf.xacro"/>
     <xacro:chassis/>
     <xacro:leg suffix="fl" parent="chassis_link" xyz="0.15 0.09 0.03" rpy="0 0.523 0"/>
@@ -15,6 +15,6 @@
     <xacro:wheel suffix="rl" parent="leg_rl" xyz="-0.08 0.02 -0.05" />
     <xacro:wheel suffix="rr" parent="leg_rr" xyz="-0.08 -0.02 -0.05" />
-    <xacro:lidar xyz="0.07 0 0.12" />
+    <xacro:display xyz="0.07 0 0.12" />
     <xacro:camera/>
-    <xacro:include filename="$(find hitomi)/urdf/gazebo_plugins.urdf.xacro"/>
+    <xacro:include filename="$(find hitomi_display)/urdf/gazebo_plugins.urdf.xacro"/>
 </robot>

File: urdf/gazebo_plugins.urdf.xacro (robot description, xacro)
@@ -29,15 +29,4 @@
   </plugin>
 </gazebo>
-<!--gazebo>
-  <plugin filename="gz-sim-diff-drive-system" name="gz::sim::systems::DiffDrive">
-      <left_joint>wheel_fl_joint</left_joint>
-      <right_joint>wheel_fr_joint</right_joint>
-      <wheel_separation>0.220334</wheel_separation>
-      <wheel_radius>0.02</wheel_radius>
-      <max_linear_acceleration>5</max_linear_acceleration>
-      <odom_publish_frequency>30</odom_publish_frequency>
-      <odom_topic>odom</odom_topic>
-  </plugin>
-  </gazebo-->
 <gazebo reference="wheel_fl">
   <mu1>1.0</mu1>

File: urdf/legs.urdf.xacro (robot description, xacro)
@@ -6,5 +6,5 @@
                 <origin xyz="0 0 0" rpy="${rpy}"/>
                 <geometry>
-                    <mesh filename="package://hitomi/meshes/leg.dae"/>
+                    <mesh filename="package://hitomi_display/meshes/leg.dae"/>
                 </geometry>
                 <material name="white">
@@ -15,5 +15,5 @@
                 <origin xyz="0 0 0" rpy="${rpy}"/>
                 <geometry>
-                    <mesh filename="package://hitomi/meshes/leg.stl"/>
+                    <mesh filename="package://hitomi_display/meshes/leg.stl"/>
                 </geometry>
             </collision>
